File: Design/KineticMod.sch (EAGLE design)
At the start: 33 parts, among them P1 ALPS_RK09K_VERTICAL, P2 ALPS_RK09K_VERTICAL, P3 ALPS_RK09K_VERTICAL, P4 ALPS_RK09K_VERTICAL, Q1 AOD417, U1 PCA9685

Commit message: Updated structure
Other:
- note removed: "By J.G.Aguado"
- note removed: "R2"
Changed lines of the file:
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@@
 <?xml version="1.0" encoding="utf-8"?>
 <!DOCTYPE eagle SYSTEM "eagle.dtd">
-<eagle version="9.4.2">
+<eagle version="9.5.1">
 <drawing>
 <settings>
@@
 <layer number="59" name="tCarbon" color="7" fill="1" visible="no" active="no"/>
 <layer number="60" name="bCarbon" color="7" fill="1" visible="no" active="no"/>
+<layer number="88" name="SimResults" color="9" fill="1" visible="yes" active="yes"/>
+<layer number="89" name="SimProbes" color="9" fill="1" visible="yes" active="yes"/>
 <layer number="90" name="Modules" color="7" fill="1" visible="yes" active="yes"/>
 <layer number="91" name="Nets" color="2" fill="1" visible="yes" active="yes"/>
@@
 </classes>
 <parts>
-<part name="FRAME1" library="frames" deviceset="A4L-LOC" device=""/>
 <part name="H1" library="holes" deviceset="MOUNT-PAD-ROUND" device="3.2" value=""/>
 <part name="H2" library="holes" deviceset="MOUNT-PAD-ROUND" device="3.2" value=""/>
@@
 <part name="U$8" library="microbuilder" deviceset="GND" device=""/>
 <part name="C3" library="rcl" library_urn="urn:adsk.eagle:library:334" deviceset="CPOL-US" device="D/7343-31R" package3d_urn="urn:adsk.eagle:package:23417/2" value="470uF"/>
+<part name="FRAME1" library="SpaceDIY_symbols" deviceset="A4L-LOC" device=""/>
 </parts>
 <sheets>
 <sheet>
 <plain>
-<text x="218.44" y="15.24" size="2.54" layer="94">By J.G.Aguado</text>
 <text x="66.548" y="79.756" size="2.032" layer="102" font="vector">Pressure</text>
 <text x="63.246" y="117.348" size="2.032" layer="102" font="vector">Humidity</text>
@@
 <text x="38.1" y="152.4" size="1.778" layer="97">I2C Address =</text>
 <text x="30.48" y="144.78" size="1.778" layer="97">Open = 0 / Closed = 1</text>
-<text x="248.92" y="5.08" size="2.54" layer="94">R2</text>
 </plain>
 <instances>
-<instance part="FRAME1" gate="G$1" x="0" y="0" smashed="yes">
-<attribute name="DRAWING_NAME" x="168.91" y="12.7" size="5.08" layer="94" font="vector"/>
-<attribute name="LAST_DATE_TIME" x="217.17" y="10.16" size="2.286" layer="94" font="vector"/>
-<attribute name="SHEET" x="230.505" y="5.08" size="2.54" layer="94" font="vector"/>
-</instance>
 <instance part="H1" gate="G$1" x="231.14" y="96.52" smashed="yes" rot="R90">
 <attribute name="NAME" x="230.5558" y="99.314" size="1.778" layer="95" rot="R90"/>
@@
 <attribute name="VALUE" x="222.504" y="46.609" size="1.778" layer="96" rot="MR0"/>
 </instance>
+<instance part="FRAME1" gate="G$1" x="0" y="0" smashed="yes">
+<attribute name="LAST_DATE_TIME" x="217.17" y="10.16" size="2.286" layer="94"/>
+<attribute name="SHEET" x="227.965" y="5.08" size="2.54" layer="94"/>
+<attribute name="DRAWING_NAME" x="217.17" y="20.32" size="2.54" layer="94"/>
+</instance>
 </instances>
